File: kicad/Eurorack_Electric_Druid_VCDO1_Control_Board.kicad_sch (KiCad schematic)
At the start: 31 parts, among them J10 Glide_time_CV_in, J11 Bitcrush_CV_in, J3 Main_osc_out, J4 Sub_osc_out, J5 Glide_on_off_CV_in, J6 Note_CV_in, J7 FM_CV_in, J8 WaveSel_CV_in, J9 SubSel_CV_in

Commit message: updated schematic rev0.1.3
Connections:
- net CB_+5V: now also RV10.3, RV14.3, RV15.3, RV7.3, RV8.3, RV9.3; no longer RV10.1, RV7.1, RV8.1, RV9.1
- net CB_-5V: no longer RV14.1, RV15.1
- net CB_GND: now also RV10.1, RV14.1, RV15.1, RV7.1, RV8.1, RV9.1; no longer RV10.3, RV14.3, RV15.3, RV7.3, RV8.3, RV9.3
Other:
- note removed: "Pots inverted on purpose!"
Changed lines of the file:
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@@
   (title_block
     (title "Eurorack Electric Druid VCDO1 - Control Board")
-    (date "2023-12-30")
-    (rev "0.1.2")
+    (date "2024-02-24")
+    (rev "0.1.3")
     (company "DIYSynthMNL")
     (comment 1 "Shared under a CC BY-NC-SA 4.0 license. Some rights reserved.")
@@
     (effects (font (size 1.27 1.27)) (justify left bottom))
   )
-  (text "Pots inverted on purpose!" (at 99.06 59.69 0)
-    (effects (font (size 1.27 1.27)) (justify left bottom))
-  )
   (text "0V-5V" (at 72.39 22.86 0)
     (effects (font (size 1.27 1.27)) (justify left bottom))
@@
     (effects (font (size 1.27 1.27)) (justify left bottom))
   )
-  (label "CB_-5V" (at 40.005 104.14 0) (fields_autoplaced)
-    (effects (font (size 1.27 1.27)) (justify left bottom))
-  )
-  (label "CB_-5V" (at 39.37 144.145 0) (fields_autoplaced)
+  (label "CB_+5V" (at 40.005 104.14 0) (fields_autoplaced)
+    (effects (font (size 1.27 1.27)) (justify left bottom))
+  )
+  (label "CB_+5V" (at 39.37 144.145 0) (fields_autoplaced)
     (effects (font (size 1.27 1.27)) (justify left bottom))
   )
@@
     )
   )
-  (symbol (lib_id "Device:R_Potentiometer") (at 31.115 100.33 0) (mirror x) (unit 1)
-    (in_bom yes) (on_board yes) (dnp no)
-    (property "Reference" "RV15" (at 28.575 99.06 0)
-      (effects (font (size 1.27 1.27)) (justify right))
-    )
-    (property "Value" "10K_Bitcrush_Control" (at 41.91 106.045 0)
+  (symbol (lib_id "Device:R_Potentiometer") (at 31.115 100.33 0) (unit 1)
+    (in_bom yes) (on_board yes) (dnp no)
+    (property "Reference" "RV15" (at 28.575 101.6 0)
+      (effects (font (size 1.27 1.27)) (justify right))
+    )
+    (property "Value" "10K_Bitcrush_Control" (at 41.275 105.41 0)
       (effects (font (size 1.27 1.27)) (justify right))
     )
@@
     )
   )
-  (symbol (lib_id "Device:R_Potentiometer") (at 167.64 98.425 0) (unit 1)
-    (in_bom yes) (on_board yes) (dnp no)
-    (property "Reference" "RV10" (at 165.1 99.695 0)
-      (effects (font (size 1.27 1.27)) (justify right))
-    )
-    (property "Value" "10K_SubWaveSel" (at 165.1 97.155 0)
+  (symbol (lib_id "Device:R_Potentiometer") (at 167.64 98.425 0) (mirror x) (unit 1)
+    (in_bom yes) (on_board yes) (dnp no)
+    (property "Reference" "RV10" (at 165.1 97.155 0)
+      (effects (font (size 1.27 1.27)) (justify right))
+    )
+    (property "Value" "10K_SubWaveSel" (at 165.1 99.695 0)
       (effects (font (size 1.27 1.27)) (justify right))
     )
@@
     )
   )
-  (symbol (lib_id "Device:R_Potentiometer") (at 167.64 67.31 0) (unit 1)
-    (in_bom yes) (on_board yes) (dnp no)
-    (property "Reference" "RV8" (at 165.1 68.58 0)
-      (effects (font (size 1.27 1.27)) (justify right))
-    )
-    (property "Value" "10K_Freq_Fine" (at 165.1 66.04 0)
+  (symbol (lib_id "Device:R_Potentiometer") (at 167.64 67.31 0) (mirror x) (unit 1)
+    (in_bom yes) (on_board yes) (dnp no)
+    (property "Reference" "RV8" (at 165.1 66.04 0)
+      (effects (font (size 1.27 1.27)) (justify right))
+    )
+    (property "Value" "10K_Freq_Fine" (at 165.1 68.58 0)
       (effects (font (size 1.27 1.27)) (justify right))
     )
@@
     )
   )
-  (symbol (lib_id "Device:R_Potentiometer") (at 120.65 67.945 0) (unit 1)
-    (in_bom yes) (on_board yes) (dnp no)
-    (property "Reference" "RV7" (at 118.11 69.215 0)
-      (effects (font (size 1.27 1.27)) (justify right))
-    )
-    (property "Value" "10K_Freq_Course" (at 118.11 66.675 0)
+  (symbol (lib_id "Device:R_Potentiometer") (at 120.65 67.945 0) (mirror x) (unit 1)
+    (in_bom yes) (on_board yes) (dnp no)
+    (property "Reference" "RV7" (at 118.11 66.675 0)
+      (effects (font (size 1.27 1.27)) (justify right))
+    )
+    (property "Value" "10K_Freq_Course" (at 118.11 69.215 0)
       (effects (font (size 1.27 1.27)) (justify right))
     )
@@
     )
   )
-  (symbol (lib_id "Device:R_Potentiometer") (at 120.65 99.06 0) (unit 1)
-    (in_bom yes) (on_board yes) (dnp no)
-    (property "Reference" "RV9" (at 118.11 100.33 0)
-      (effects (font (size 1.27 1.27)) (justify right))
-    )
-    (property "Value" "10K_MainWaveSel" (at 118.11 97.79 0)
+  (symbol (lib_id "Device:R_Potentiometer") (at 120.65 99.06 0) (mirror x) (unit 1)
+    (in_bom yes) (on_board yes) (dnp no)
+    (property "Reference" "RV9" (at 118.11 97.79 0)
+      (effects (font (size 1.27 1.27)) (justify right))
+    )
+    (property "Value" "10K_MainWaveSel" (at 118.11 100.33 0)
       (effects (font (size 1.27 1.27)) (justify right))
     )
@@
     )
   )
-  (symbol (lib_id "Device:R_Potentiometer") (at 31.75 140.335 0) (mirror x) (unit 1)
-    (in_bom yes) (on_board yes) (dnp no)
-    (property "Reference" "RV14" (at 29.21 139.065 0)
-      (effects (font (size 1.27 1.27)) (justify right))
-    )
-    (property "Value" "10K_GlideTime_Control" (at 41.91 145.415 0)
-      (effects (font (size 1.27 1.27)) (justify right))
-    )
+  (symbol (lib_id "Device:R_Potentiometer") (at 31.75 140.335 0) (unit 1)
+    (in_bom yes) (on_board yes) (dnp no)
+    (property "Reference" "RV14" (at 29.21 141.605 0)
+      (effects (font (size 1.27 1.27)) (justify right))
+    )
+    (property "Value" "10K_GlideTime_Control" (at 42.545 145.415 0)
+      (effects (font (size 1.27 1.27)) (justify right))
+    )
