File: kicad/Eurorack_Electric_Druid_VCDO1_Front_Panel.kicad_sch (KiCad schematic)
At the start: 0 parts

Commit message: updated schematic rev0.1.3
Other:
- title: Eurorack Electric Druid VCDO1 - Front Panel -> Eurorack Electric Druid VCDO1 - Control Board
Changed lines of the file:
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@@
   (paper "A4")
   (title_block
-    (title "Eurorack Electric Druid VCDO1 - Front Panel")
-    (date "2023-12-30")
-    (rev "0.1.2")
+    (title "Eurorack Electric Druid VCDO1 - Control Board")
+    (date "2024-02-24")
+    (rev "0.1.3")
     (company "DIYSynthMNL")
     (comment 1 "Shared under a CC BY-NC-SA 4.0 license. Some rights reserved.")
